File: hardware/KiCad/windmeter-modbus-interface.kicad_pcb (KiCad board)
At the start: 2 copper layers, 4 parts, among them U1 CH32V003J4M6, U2 MAX3485, U3 CH32V003A4M6, U4 CH32V003F4P6

Commit message: Update PCB
Parts:
- removed U3: CH32V003A4M6, Package_SO:STC_SOP-16_3.9x9.9mm_P1.27mm
- removed U4: CH32V003F4P6, Package_SO:TSSOP-20_4.4x6.5mm_P0.65mm
- added C1: 100n, Capacitor_SMD:C_1206_3216Metric_Pad1.33x1.80mm_HandSolder, F.Cu at (144.9, 127.3)
- added C2: 100n, Capacitor_SMD:C_1206_3216Metric_Pad1.33x1.80mm_HandSolder, F.Cu at (144.9, 130.6)
- added D1: SM712_SOT23, Package_TO_SOT_SMD:SOT-23, F.Cu at (144.4, 134.5)
- added J1: MODBUS-P1, my-KiCad-library:CONN_215877-1, F.Cu at (137.1, 116.9)
- added J2: Programming, Connector_PinHeader_2.54mm:PinHeader_1x03_P2.54mm_Vertical, F.Cu at (135.3, 127.9)
- added J3: MODBUS-P2, my-KiCad-library:CONN_215877-1, F.Cu at (156.3, 116.9)
- added JP1: enable term., Jumper:SolderJumper-2_P1.3mm_Open_Pad1.0x1.5mm, F.Cu at (139.7, 127.4)
- added JP2: ~, Jumper:SolderJumper-3_P1.3mm_Bridged12_Pad1.0x1.5mm_NumberLabels, F.Cu at (117.1, 124.7)
- added JP3: ~, Jumper:SolderJumper-3_P1.3mm_Bridged12_Pad1.0x1.5mm_NumberLabels, F.Cu at (117.1, 128.6)
- added JP4: ~, Jumper:SolderJumper-3_P1.3mm_Bridged12_Pad1.0x1.5mm_NumberLabels, F.Cu at (117.1, 132.4)
- added JP5: ~, Jumper:SolderJumper-3_P1.3mm_Bridged12_Pad1.0x1.5mm_NumberLabels, F.Cu at (117.1, 136.2)
- added JP6: Address select, Jumper:SolderJumper-2_P1.3mm_Open_Pad1.0x1.5mm, F.Cu at (139.7, 130.9)
- added R1: 120, Resistor_SMD:R_1206_3216Metric_Pad1.30x1.75mm_HandSolder, F.Cu at (130.0, 127.2)
- added R2: 20k, Resistor_SMD:R_1206_3216Metric_Pad1.30x1.75mm_HandSolder, F.Cu at (130.0, 130.5)
- added R3: 20k, Resistor_SMD:R_1206_3216Metric_Pad1.30x1.75mm_HandSolder, F.Cu at (130.0, 133.9)
- added R4: 10k, Resistor_SMD:R_1206_3216Metric_Pad1.30x1.75mm_HandSolder, F.Cu at (130.0, 137.2)
Connections:
- U1 pad 1: unconnected-(U1-PD6/PA1-Pad1) -> /MB-TX/RX
- U1 pad 2: unconnected-(U1-VSS-Pad2) -> /GND
- U1 pad 3: unconnected-(U1-PA2-Pad3) -> /ANALOG_IN
- U1 pad 4: unconnected-(U1-VDD-Pad4) -> /3V3
- U1 pad 5: unconnected-(U1-PC1-Pad5) -> /PULSE_IN
- U1 pad 6: unconnected-(U1-PC2-Pad6) -> /MB-RE/DE
- U1 pad 7: unconnected-(U1-PC4-Pad7) -> /ADDRESS
- U1 pad 8: unconnected-(U1-PD1/PD4/PD5-Pad8) -> /SWIO
- U2 pad 1: unconnected-(U2-RO-Pad1) -> /MB-TX/RX
- U2 pad 2: unconnected-(U2-~{RE}-Pad2) -> /MB-RE/DE
- U2 pad 3: unconnected-(U2-DE-Pad3) -> /MB-RE/DE
- U2 pad 4: unconnected-(U2-DI-Pad4) -> /MB-TX/RX
- U2 pad 5: unconnected-(U2-GND-Pad5) -> /GND
- U2 pad 6: unconnected-(U2-A-Pad6) -> /RS485-A
- U2 pad 7: unconnected-(U2-B-Pad7) -> /RS485-B
- U2 pad 8: unconnected-(U2-VCC-Pad8) -> /3V3
