File: hardware/KiCad/windmeter-modbus-interface.kicad_pcb (KiCad board)
At the start: 2 copper layers, 18 parts, among them J1 MODBUS-P1, J2 Programming, J3 MODBUS-P2, U1 CH32V003J4M6, U2 MAX3485

Commit message: Update PCB Design
Parts:
- added B1: DB207, my-KiCad-library:DB207, F.Cu at (128.3, 145.2)
- added C3: 100u, Capacitor_THT:CP_Radial_D8.0mm_P5.00mm, F.Cu at (124.2, 135.4)
- added C4: 4u7, Capacitor_THT:CP_Radial_D5.0mm_P2.50mm, F.Cu at (109.9, 135.4)
- added C5: 100n, Capacitor_SMD:C_1206_3216Metric_Pad1.33x1.80mm_HandSolder, F.Cu at (119.8, 108.8)
- added D2: BZX84Cxx, Package_TO_SOT_SMD:SOT-23, F.Cu at (124.5, 108.8)
- added J4: RJ14, Connector_RJ:RJ14_Connfly_DS1133-S4_Horizontal, F.Cu at (109.0, 98.8)
- added J5: RJ14, Connector_RJ:RJ14_Connfly_DS1133-S4_Horizontal, F.Cu at (125.5, 98.8)
- added P1: ~, my-KiCad-library:HLK-K7803-500R3, F.Cu at (112.5, 143.4)
- added R5: 10k, Resistor_SMD:R_1206_3216Metric_Pad1.30x1.75mm_HandSolder, F.Cu at (111.9, 108.8)
- added R6: 100, Resistor_SMD:R_1206_3216Metric_Pad1.30x1.75mm_HandSolder, F.Cu at (115.8, 108.8)
- added R7: 10k, Resistor_SMD:R_1206_3216Metric_Pad1.30x1.75mm_HandSolder, F.Cu at (109.9, 117.6)
- JP1, JP2, JP3, JP4, JP5, JP6: moved to B.Cu
- moved J1 61.6 mm to (109.7, 172.1)
- moved J3 61.6 mm to (128.9, 172.1)
- moved C1 35.0 mm to (109.9, 127.1)
- moved R1 33.8 mm to (115.2, 157.6), turned to 180 degrees
- moved JP2 33.7 mm to (109.2, 157.5), turned to 180 degrees
- moved R3 33.0 mm to (107.1, 157.6)
- moved JP1 32.8 mm to (118.9, 152.7)
- moved D1 31.6 mm to (122.8, 157.6)
- moved U1 30.1 mm to (120.7, 122.6)
- moved JP4 27.5 mm to (128.4, 157.5), turned to 180 degrees
- moved R2 27.1 mm to (130.5, 157.6)
- moved JP3 25.4 mm to (109.2, 152.7), turned to 180 degrees
- moved C2 24.4 mm to (120.7, 127.1)
- moved JP5 19.9 mm to (128.4, 152.7), turned to 180 degrees
- moved JP6 14.9 mm to (127.4, 122.5), turned to 90 degrees
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Connections:
- net /24V renamed /+24V
- J1 pad 7: /GND -> /-24V
- J1 pad 8: /GND -> /-24V
- J3 pad 7: /GND -> /-24V
- J3 pad 8: /GND -> /-24V
Routing:
- net /3V3: track 0.00 -> 99.1 mm
- net /GND: track 0.00 -> 71.1 mm, vias 0 -> 2
- net /+24V: track 0.00 -> 49.2 mm
- net /-24V: track 0.00 -> 45.3 mm
- net Net-(P1-GND): track 0.00 -> 37.9 mm
- net /RS485-A: track 0.00 -> 34.6 mm, vias 0 -> 4
- net /RS485-B: track 0.00 -> 30.9 mm, vias 0 -> 3
- net /MB-RE/DE: track 0.00 -> 27.8 mm
- net /Ba: track 0.00 -> 24.7 mm
- net /_Ba: track 0.00 -> 24.7 mm
- net Net-(P1-IN): track 0.00 -> 16.5 mm
- net /_Bb: track 0.00 -> 14.8 mm
- net /Bb: track 0.00 -> 14.7 mm
- net /PULSE_IN: track 0.00 -> 14.2 mm
- net /MB-TX/RX: track 0.00 -> 12.1 mm
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