File: hardware/KiCad/windmeter-modbus-interface.kicad_pcb (KiCad board)
At the start: 2 copper layers, 70 x 92 mm, 30 parts, among them J1 MODBUS-P1, J2 Programming, J3 MODBUS-P2, J4 RJ14, J5 RJ14, U1 CH32V003J4M6, U2 MAX3485

Commit message: Updated text on PCB design
Other:
- board text added: "Modbus-RS485 Port-1"
- board text added: "Modbus-RS485 Port-2"
- board text added: "Wind-speed/-direction to Modbus RTU RS-485 interface"
- board text added: "modbus-termination, RS485 pair selection & Address at back of PCB."
- board text removed: "MODBus-RS458 Port-1"
- board text removed: "MODBus-RS458 Port-2"
- board text removed: "Wind-speed/-direction to modbus interface"
- board text removed: "modbus-termination, RS458 pair selection & Address at back of PCB."
Changed lines of the file:
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@@
 		(layer "Edge.Cuts")
 	)
-	(gr_text "modbus-termination, \nRS458 pair selection &\nAddress at back of PCB."
+	(gr_text "modbus-termination, \nRS485 pair selection &\nAddress at back of PCB."
 		(at 155.194 63.881 0)
 		(layer "F.SilkS" knockout)
@@
 		)
 	)
-	(gr_text "MODBus-RS458\nPort-2"
+	(gr_text "Modbus-RS485\nPort-2"
 		(at 207.518 132.461 0)
 		(layer "F.SilkS")
@@
 		)
 	)
-	(gr_text "MODBus-RS458\nPort-1"
+	(gr_text "Modbus-RS485\nPort-1"
 		(at 168.402 132.461 0)
 		(layer "F.SilkS")
@@
 		)
 	)
-	(gr_text "Wind-speed/-direction to\nmodbus interface"
+	(gr_text "Wind-speed/-direction to\nModbus RTU RS-485 interface"
 		(at 210.947 128.651 90)
 		(layer "F.SilkS")
