File: hardware/KiCad/windmeter-modbus-interface.kicad_sch (KiCad schematic)
At the start: 27 parts, among them J1 MODBUS-P1, J2 Programming, J3 MODBUS-P2, J4 RJ14, U1 CH32V003J4M6, U2 MAX3485

Commit message: Modbus RTU driver: 26/26 TDS matrix on TTL rig; zero-ISR architecture
software/drivers/modbus_rtu/ (new)
- Slave driver implementing the TDS 2 layer: framing/CRC, t3.5 gap
  detect, address/broadcast filtering, FC03/04/06/16, exceptions
  01/02/03, no-clamp rejection, atomic FC16, quantity/bytecount
  validation, big-endian data + LE CRC, FC06 echo / FC16 confirm,
  app-owned register table with min/max + cross-validate hook (FR-S31)
- HIL (M2K as open-drain bit-banged master, no transceiver yet):
  26/26 vectors, 40/40 endurance, latency median/worst 5.2 ms
- Diagnostics registers: CRC/served/FE/NE/ORE counters + last-bad-frame
  stash (decisive in both bench hunts)

Two bench-forced design changes (recorded in softwareArchitecture.md,
driver README, scratchBook):
- HDSEL abandoned: intermittently swallows the first RX byte after bus
  idle (~35%, no error flags, wire pristine). Replaced by remap
  switching: RX natively on PD6 (default map), TX remapped onto PD6
  only while transmitting the response. Self-echo eliminated.
- Interrupts abandoned: RXNE ISR corrupted ~1/3 of frames (suspected
  interrupt prologue issue on this RV32EC toolchain path). Polled RX is
  provably lossless (1 us loop vs 1042 us/byte); architecture is now
  zero-ISR with no concurrency surface at all.

software/hil/
- mb_check.py: 26-vector matrix mapped to FR-MB IDs
- saleae_serial.py: raw-edge software UART decoder (Logic 2 Async
  Serial analyzer scrambles bytes at 9600) + binary-safe decode option
- README: Modbus TTL-rig lessons (M2K open-drain master, phantom start
  bits, immediate wire release, analyzer workaround)

hardware/KiCad/
- Add 10k pull-down on MB-RE/DE: holds the MAX3485 in receive mode
  while the MCU is in reset / being flashed (floating DE could jam the
  shared bus). Verified A/B fail-safe bias orientation (R2 A->3V3,
  R3 B->GND). Existing DI+RO / DE+RE ties confirmed compatible with the
  remap-switching discipline - no other PCB change needed.

design/: plan 5 exit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
Parts:
- added R7: 10k, Resistor_SMD:R_1206_3216Metric_Pad1.30x1.75mm_HandSolder, symbol Device:R
Connections:
- net GND: now also R7.2
- net MB-RE/DE: now also R7.1
Changed lines of the file:
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@@
 	)
 	(junction
+		(at 54.61 90.17)
+		(diameter 0)
+		(color 0 0 0 0)
+	)
+	(junction
 		(at 91.44 109.22)
 		(diameter 0)
@@
 	)
 	(junction
+		(at 54.61 109.22)
+		(diameter 0)
+		(color 0 0 0 0)
+	)
+	(junction
 		(at 59.69 87.63)
 		(diameter 0)
@@
 	(wire
 		(pts
+			(xy 54.61 90.17) (xy 62.23 90.17)
+		)
+		(stroke
+			(width 0)
+			(type default)
+		)
+	)
+	(wire
+		(pts
 			(xy 219.71 74.93) (xy 217.17 74.93)
 		)
@@
 	(wire
 		(pts
-			(xy 45.72 90.17) (xy 62.23 90.17)
+			(xy 45.72 90.17) (xy 54.61 90.17)
 		)
 		(stroke
@@
 	(wire
 		(pts
+			(xy 54.61 90.17) (xy 54.61 99.06)
+		)
+		(stroke
+			(width 0)
+			(type default)
+		)
+	)
+	(wire
+		(pts
 			(xy 64.77 38.1) (xy 64.77 54.61)
 		)
@@
 	(wire
 		(pts
+			(xy 54.61 106.68) (xy 54.61 109.22)
+		)
+		(stroke
+			(width 0)
+			(type default)
+		)
+	)
+	(wire
+		(pts
+			(xy 54.61 109.22) (xy 64.77 109.22)
+		)
+		(stroke
+			(width 0)
+			(type default)
+		)
+	)
+	(wire
+		(pts
 			(xy 64.77 30.48) (xy 64.77 29.21)
 		)
@@
 	(wire
 		(pts
-			(xy 45.72 109.22) (xy 64.77 109.22)
+			(xy 45.72 109.22) (xy 54.61 109.22)
 		)
 		(stroke
@@
 					(unit 1)
 				)
+			)
+		)
+	)
+	(symbol
+		(lib_id "Device:R")
+		(at 54.61 102.87 0)
+		(unit 1)
+		(body_style 1)
+		(exclude_from_sim no)
+		(in_bom yes)
+		(on_board yes)
+		(in_pos_files yes)
+		(dnp no)
+		(fields_autoplaced yes)
+		(property "Reference" "R7"
+			(at 57.15 101.5999 0)
+			(show_name no)
+			(do_not_autoplace no)
+			(effects
+				(font
+					(size 1.27 1.27)
+				)
+				(justify left)
+			)
+		)
+		(property "Value" "10k"
+			(at 57.15 104.1399 0)
+			(show_name no)
+			(do_not_autoplace no)
+			(effects
+				(font
+					(size 1.27 1.27)
+				)
+				(justify left)
+			)
+		)
+		(property "Footprint" "Resistor_SMD:R_1206_3216Metric_Pad1.30x1.75mm_HandSolder"
+			(at 52.832 102.87 90)
+			(hide yes)
+			(show_name no)
+			(do_not_autoplace no)
+			(effects
+				(font
+					(size 1.27 1.27)
+				)
+			)
+		)
+		(property "Datasheet" ""
+			(at 54.61 102.87 0)
+			(hide yes)
+			(show_name no)
+			(do_not_autoplace no)
+			(effects
+				(font
+					(size 1.27 1.27)
+				)
+			)
+		)
+		(property "Description" "Resistor"
+			(at 54.61 102.87 0)
+			(hide yes)
+			(show_name no)
+			(do_not_autoplace no)
+			(effects
+				(font
+					(size 1.27 1.27)
+				)
+			)
+		)
+		(pin "1"
+		)
+		(pin "2"
+		)
+		(instances
+			(project "windmeter-modbus-interface"
+				(path "/7e9d7b84-ea76-433c-8a90-337ecd1345cc"
+					(reference "R7")
+					(unit 1)
+				)
