File: hardware/KiCad/windmeter-modbus-interface.kicad_sch (KiCad schematic)
At the start: 28 parts, among them J1 MODBUS-P1, J2 Programming, J3 MODBUS-P2, J4 RJ14, U1 CH32V003J4M6, U2 MAX3485

Commit message: Update PCB Design
Parts:
- added J5: RJ14, Connector_RJ:RJ14_Connfly_DS1133-S4_Horizontal, symbol Connector:RJ14
- B1: footprint DB207:DB207 -> my-KiCad-library:DB207
- C3: footprint (none) -> Capacitor_THT:CP_Radial_D8.0mm_P5.00mm
- C4: footprint (none) -> Capacitor_THT:CP_Radial_D5.0mm_P2.50mm
- J4: footprint (none) -> Connector_RJ:RJ14_Connfly_DS1133-S4_Horizontal
- P1: footprint (none) -> my-KiCad-library:HLK-K7803-500R3
Connections:
- net 3V3: now also J5.1
- net ANALOG_IN: now also J5.4; no longer J4.4
- net GND: now also J5.3; no longer B1.AC2 (~@2), J1.7 (8), J1.8 (7), J3.7 (8), J3.8 (7)
- net 24V renamed +24V
- new net -24V: B1.AC2 (~@2), J1.7 (8), J1.8 (7), J3.7 (8), J3.8 (7)
Other:
- note added: "Wind- direction"
- note added: "Wind- speed"
- moved on the sheet: C5, D2, J1, J2, J3, J4, JP2, JP3, JP4, JP5, R5, R6
