File: hardware/KiCad/windmeter-modbus-interface.kicad_sch (KiCad schematic)
At the start: 29 parts, among them J1 MODBUS-P1, J2 Programming, J3 MODBUS-P2, J4 RJ14, J5 RJ14, U1 CH32V003J4M6, U2 MAX3485

Commit message: Repository documentation: README, changelog, contributing, licenses
Root docs adapted from the tester-repo templates to this project:
- README: device overview, variant/address table, project status with
  pointers into the design chain, hardware summary, register-map summary,
  repo layout, build/flash/test instructions (incl. acceptance suite and
  submodule clone), related repositories
- changelog: project history to date under [Unreleased] (design chain,
  TDS v0.6, drivers with HIL results, firmware stages A-F, HIL harness);
  release tagging deferred to RELEASES.md's fw-v<N> process
- contributing: correct repo URL, requirements-first workflow (TDS IDs),
  build/test expectations, *_test binaries never released
- LICENSE/license.md: project name corrected; third-party section names
  the actual manufacturers and covers the KiCad library submodules

Co-Authored-By: Claude Fable 5 <noreply@anthropic.com>
Parts:
- B1: footprint my-KiCad-library:DB207 -> my-KiCad-library:DB207-DIP-4
Connections:
- net GND: now also B1.-, C3.2, C4.2, P1.2 (GND)
Changed lines of the file:
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@@
 	)
 	(junction
+		(at 111.76 181.61)
+		(diameter 0)
+		(color 0 0 0 0)
+	)
+	(junction
 		(at 222.25 104.14)
 		(diameter 0)
@@
 	(wire
 		(pts
+			(xy 111.76 181.61) (xy 123.19 181.61)
+		)
+		(stroke
+			(width 0)
+			(type default)
+		)
+	)
+	(wire
+		(pts
 			(xy 176.53 45.72) (xy 187.96 45.72)
 		)
@@
 		)
 	)
+	(label "GND"
+		(at 121.92 181.61 180)
+		(effects
+			(font
+				(size 1.27 1.27)
+			)
+			(justify right bottom)
+		)
+	)
 	(label "+24V"
 		(at 46.99 161.29 0)
@@
 			)
 		)
-		(property "Footprint" "my-KiCad-library:DB207"
+		(property "Footprint" "my-KiCad-library:DB207-DIP-4"
 			(at 42.164 139.7 0)
 			(hide yes)

Commit message: TDS v0.9: promote as-built hardware (§4) from KiCad; resolve open items
Add §4 Hardware sourced from the as-built KiCad PCB — normative MCU
pin/net map, RS-485 front-end, 24V PoE power chain, sensor front-ends,
connectors, and the anemometer calibration derivation. Renumber NFRs→§5,
Open items→§6.

Walk through and close/narrow the §6 open items: response latency measured
(4-5 ms), temperature range bounded by as-built parts, direction accuracy
firmware-closed, volatile-register and combined-variant decisions recorded.
Reconcile stale notes with the shipped firmware: FR-MB23 remap-switching
(not HDSEL), FR-S27 pulses-per-rotation now runtime-configurable (FR-S40).

Record as-built deltas vs scratchBook (fail-safe R2/R3 designators, power
caps 100uF/4.7uF, two RJ14 jacks, no ADC RC filter, unspecified zener,
RS458 silk typo). Sync README/design-README to v0.9; changelog entry.

Co-Authored-By: Claude Opus 4.8 <noreply@anthropic.com>
Parts:
- D2: value BZX84Cxx -> BZX84-C3V3
Other:
- title: Windmeter interface for Modbus RS458 -> Windmeter interface for Modbus RS485
Changed lines of the file:
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@@
 	(paper "A4")
 	(title_block
-		(title "Windmeter interface for Modbus RS458")
+		(title "Windmeter interface for Modbus RS485")
 		(date "2026-06-28")
 		(company "RFSee")
@@
 			)
 		)
-		(property "Value" "BZX84Cxx"
+		(property "Value" "BZX84-C3V3"
 			(at 212.09 93.9799 90)
 			(show_name no)
